File: pcb/conndom.kicad_sch (KiCad schematic)
At the start: 17 parts, among them J1 USB C PWR, J2 USB A WIFI

Commit message: bom for PCBWay WiP
Parts:
- C1, R1, R2, R3, R4: Package (none) -> 0805; Type (none) -> SMD
- J1: value USB C PWR -> UJC-HP2-3-SMT-TR; MANUFACTURER CUI Devices -> (none); MAXIMUM_PACKAGE_HEIGHT 3.16mm -> (none); PARTREV 1.01 -> (none); STANDARD Manufacturer Recommendations -> (none)
- J2: value USB A WIFI -> UJ2-AH-4-TH; MANUFACTURER CUI INC -> (none); PART_REV 1.0 -> (none); STANDARD MANUFACTURER RECOMMENDATIONS -> (none)
- S1: value PWR -> TS02-66-55-BK-260-LCR-D; MANUFACTURER CUI Devices -> (none); PARTREV 1.0 -> (none); STANDARD Manufacturer Recommendations -> (none)

Commit message: updates values in BOM
Parts:
- C1: value 104 -> 104n; Package 0805 -> (none); Type SMD -> (none)
- D1: Type (none) -> SMD
- J1: Manufacturer (none) -> Same Sky; Mfg Part # (none) -> UJC-HP2-3-SMT-TR; Type (none) -> SMD/THT
- J2: Manufacturer (none) -> Same Sky; Mfg Part # (none) -> UJ2-AH-4-TH; Type (none) -> SMD/THT
- R4: value 10k -> 10K
- S1: Manufacturer (none) -> Same Sky; Mfg Part # (none) -> TS02-66-55-BK-260-LCR-D; Type (none) -> THT
Changed lines of the file:
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@@
 			)
 		)
-		(property "Value" "104"
+		(property "Value" "104n"
 			(at 220.98 123.1899 0)
 			(effects
@@
 			)
 		)
-		(property "Datasheet" "~"
+		(property "Datasheet" ""
 			(at 217.17 121.92 0)
 			(effects
@@
 			)
 		)
-		(property "Manufacturer" "~"
+		(property "Manufacturer" ""
 			(at 217.17 121.92 0)
 			(effects
@@
 			)
 		)
-		(property "Mfg Part #" "~"
+		(property "Mfg Part #" ""
 			(at 217.17 121.92 0)
 			(effects
@@
 			)
 		)
-		(property "Package" "0805"
+		(property "Package" ""
 			(at 217.17 121.92 0)
 			(effects
@@
 			)
 		)
-		(property "Type" "SMD"
+		(property "Type" ""
 			(at 217.17 121.92 0)
 			(effects
@@
 			)
 		)
-		(property "Manufacturer" ""
+		(property "Manufacturer" "Same Sky"
 			(at 96.52 107.95 0)
 			(effects
@@
 			)
 		)
-		(property "Mfg Part #" ""
+		(property "Mfg Part #" "UJ2-AH-4-TH"
 			(at 96.52 107.95 0)
 			(effects
@@
 			)
 		)
-		(property "Package" ""
+		(property "Package" "~"
 			(at 96.52 107.95 0)
 			(effects
@@
 			)
 		)
-		(property "Type" ""
+		(property "Type" "SMD/THT"
 			(at 96.52 107.95 0)
 			(effects
@@
 			)
 		)
-		(property "Manufacturer" ""
+		(property "Manufacturer" "Same Sky"
 			(at 189.23 123.19 90)
 			(effects
@@
 			)
 		)
-		(property "Mfg Part #" ""
+		(property "Mfg Part #" "TS02-66-55-BK-260-LCR-D"
 			(at 189.23 123.19 90)
 			(effects
@@
 			)
 		)
-		(property "Package" ""
+		(property "Package" "~"
 			(at 189.23 123.19 90)
 			(effects
@@
 			)
 		)
-		(property "Type" ""
+		(property "Type" "THT"
 			(at 189.23 123.19 90)
 			(effects
@@
 			)
 		)
-		(property "Manufacturer" ""
+		(property "Manufacturer" "Same Sky"
 			(at 53.34 113.03 0)
 			(effects
@@
 			)
 		)
-		(property "Mfg Part #" ""
+		(property "Mfg Part #" "UJC-HP2-3-SMT-TR"
 			(at 53.34 113.03 0)
 			(effects
@@
 			)
 		)
-		(property "Package" ""
+		(property "Package" "~"
 			(at 53.34 113.03 0)
 			(effects
@@
 			)
 		)
-		(property "Type" ""
+		(property "Type" "SMD/THT"
 			(at 53.34 113.03 0)
 			(effects
@@
 			)
 		)
-		(property "Manufacturer" ""
+		(property "Manufacturer" "~"
 			(at 241.3 121.92 0)
 			(effects
@@
 			)
 		)
-		(property "Mfg Part #" ""
+		(property "Mfg Part #" "~"
 			(at 241.3 121.92 0)
 			(effects
@@
 			)
 		)
-		(property "Package" ""
+		(property "Package" "~"
 			(at 241.3 121.92 0)
 			(effects
@@
 			)
 		)
-		(property "Type" ""
+		(property "Type" "SMD"
 			(at 241.3 121.92 0)
 			(effects
@@
 			)
 		)
-		(property "Value" "10k"
+		(property "Value" "10K"
 			(at 206.502 101.6 90)
 			(effects
@@
 		(on_board yes)
 		(dnp no)
-		(fields_autoplaced yes)
 		(property "Reference" "R1"
 			(at 76.2 124.4599 0)
